File: Enclosure_02/Kicad_PCB_Plate/PCB_02/PCB_02.sch (KiCad schematic (older format))
At the start: 14 parts, among them J1 Conn_01x07_Female, J2 Conn_01x07_Female

Commit message: Update PCB_02 files
Parts:
- J1, J2: LCSC (none) -> C358721
Changed lines of the file:
@@
 F 2 "Connector:1x7_2.54mm_FemaleHeader" H 5200 3000 50  0001 C CNN
 F 3 "~" H 5200 3000 50  0001 C CNN
+F 4 "C358721" H 5200 3000 50  0001 C CNN "LCSC"
 	1    5200 3000
 	1    0    0    -1
@@
 F 2 "Connector:1x7_2.54mm_FemaleHeader" H 6400 3000 50  0001 C CNN
 F 3 "~" H 6400 3000 50  0001 C CNN
+F 4 "C358721" H 6400 3000 50  0001 C CNN "LCSC"
 	1    6400 3000
 	1    0    0    -1
